File: LrT16.kicad_sch (KiCad schematic)
At the start: 193 parts, among them J1 USB_C_Receptacle_USB2.0, J2 Conn_02x05_Odd_Even, Q1 2N7002, SW1 EC11_SMD, SW10 EC11_SMD, SW11 EC11_SMD, SW12 EC11_SMD, SW13 EC11_SMD, SW14 EC11_SMD, SW15 EC11_SMD, SW16 EC11_SMD, SW17 SW_Push, SW2 EC11_SMD, SW20 SW_SPST, SW3 EC11_SMD, SW4 EC11_SMD, SW5 EC11_SMD, SW6 EC11_SMD, SW7 EC11_SMD, SW8 EC11_SMD, SW9 EC11_SMD, U1 STM32F072C8Tx, U2 SPX3819M5-L3-3TR

Commit message: Commited for board order
Parts:
- added C37: 33n, Capacitor_SMD:C_0805_2012Metric, symbol LrE-6-rescue:C-Device
- added R56: 10K, Resistor_SMD:R_0805_2012Metric, symbol LrE-6-rescue:R-Device
- added SW18: SW_Push, LrE-6:SKHLLAA010, symbol Switch:SW_Push
Connections:
- net +3V3: now also R56.1
- net GND: now also C37.2, SW18.1
- net SW2: now reaches U1.12 (PA2)
- net SW2: now also C37.1, R56.2, SW18.2
- no-connect marks 18 -> 17
