File: LrT16.kicad_sch (KiCad schematic)
At the start: 250 parts, among them J1 USB_C_Receptacle_USB2.0, J2 Conn_02x05_Odd_Even, Q1 2N7002, Q2 2N7002, SW1 EC11_SMD, SW10 EC11_SMD, SW11 EC11_SMD, SW12 EC11_SMD, SW13 EC11_SMD, SW14 EC11_SMD, SW15 EC11_SMD, SW16 EC11_SMD, SW17 SW_Push, SW18 SW_Push, SW2 EC11_SMD, SW20 SW_SPST, SW3 EC11_SMD, SW4 EC11_SMD, SW5 EC11_SMD, SW6 EC11_SMD, SW7 EC11_SMD, SW8 EC11_SMD, SW9 EC11_SMD, U1 STM32F072C8Tx, U2 SPX3819M5-L3-3TR

Commit message: replace parts 1N4148WS to 1N4148WT due to JLCPCB message the does not fit into footprints.
Parts:
- D1, D10, D11, D12, D13, D14, D15, D16, D17, D18, D19, D2, D20, D21, D22, D23, D24, D25, D26, D27, D28, D29, D3, D30, D31, D32, D33, D34, D35, D36, D37, D38, D39, D4, D40, D41, D42, D43, D44, D45, D46, D47, D48, D5, D58, D6, D7, D8, D9: value 1N4148WS -> 1N4148WT
Changed lines of the file:
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@@
 			)
 		)
-		(property "Value" "1N4148WS"
+		(property "Value" "1N4148WT"
 			(at 461.518 129.54 0)
 			(effects
@@
 			)
 		)
-		(property "Value" "1N4148WS"
+		(property "Value" "1N4148WT"
 			(at 462.026 84.836 0)
 			(effects
@@
 			)
 		)
-		(property "Value" "1N4148WS"
+		(property "Value" "1N4148WT"
 			(at 462.026 174.752 0)
 			(effects
@@
 			)
 		)
-		(property "Value" "1N4148WS"
+		(property "Value" "1N4148WT"
 			(at 559.054 36.068 0)
 			(effects
@@
 			)
 		)
-		(property "Value" "1N4148WS"
+		(property "Value" "1N4148WT"
 			(at 561.594 83.058 0)
 			(effects
@@
 			)
 		)
-		(property "Value" "1N4148WS"
+		(property "Value" "1N4148WT"
 			(at 463.804 36.576 0)
 			(effects
@@
 			)
 		)
-		(property "Value" "1N4148WS"
+		(property "Value" "1N4148WT"
 			(at 563.118 130.81 0)
 			(effects
@@
 			)
 		)
-		(property "Value" "1N4148WS"
+		(property "Value" "1N4148WT"
 			(at 560.324 174.244 0)
 			(effects
@@
 			)
 		)
-		(property "Value" "1N4148WS"
+		(property "Value" "1N4148WT"
 			(at 294.767 90.932 0)
 			(effects
@@
 			)
 		)
-		(property "Value" "1N4148WS"
+		(property "Value" "1N4148WT"
 			(at 395.097 186.182 0)
 			(effects
@@
 			)
 		)
-		(property "Value" "1N4148WS"
+		(property "Value" "1N4148WT"
 			(at 195.707 143.002 0)
 			(effects
@@
 			)
 		)
-		(property "Value" "1N4148WS"
+		(property "Value" "1N4148WT"
 			(at 196.977 183.642 0)
 			(effects
@@
 			)
 		)
-		(property "Value" "1N4148WS"
+		(property "Value" "1N4148WT"
 			(at 393.827 42.672 0)
 			(effects
@@
 			)
 		)
-		(property "Value" "1N4148WS"
+		(property "Value" "1N4148WT"
 			(at 360.426 84.582 0)
 			(effects
@@
 			)
 		)
-		(property "Value" "1N4148WS"
+		(property "Value" "1N4148WT"
 			(at 392.557 90.932 0)
 			(effects
@@
 			)
 		)
-		(property "Value" "1N4148WS"
+		(property "Value" "1N4148WT"
 			(at 293.497 137.922 0)
 			(effects
@@
 			)
 		)
-		(property "Value" "1N4148WS"
+		(property "Value" "1N4148WT"
 			(at 490.347 141.732 0)
 			(effects
@@
 			)
 		)
-		(property "Value" "1N4148WS"
+		(property "Value" "1N4148WT"
 			(at 490.347 46.482 0)
 			(effects
@@
 			)
 		)
-		(property "Value" "1N4148WS"
+		(property "Value" "1N4148WT"
 			(at 360.68 131.318 0)
 			(effects
@@
 			)
 		)
-		(property "Value" "1N4148WS"
+		(property "Value" "1N4148WT"
 			(at 293.497 47.752 0)
 			(effects
@@
 			)
 		)
-		(property "Value" "1N4148WS"
+		(property "Value" "1N4148WT"
 			(at 489.077 186.182 0)
 			(effects
@@
 			)
 		)
-		(property "Value" "1N4148WS"
+		(property "Value" "1N4148WT"
 			(at 489.077 181.102 0)
 			(effects
@@
 			)
 		)
-		(property "Value" "1N4148WS"
+		(property "Value" "1N4148WT"
 			(at 196.977 188.722 0)
 			(effects
@@
 			)
 		)
-		(property "Value" "1N4148WS"
+		(property "Value" "1N4148WT"
 			(at 195.707 137.922 0)
 			(effects
@@
 			)
 		)
-		(property "Value" "1N4148WS"
+		(property "Value" "1N4148WT"
 			(at 490.347 89.662 0)
 			(effects
@@
 			)
 		)
-		(property "Value" "1N4148WS"
+		(property "Value" "1N4148WT"
 			(at 293.497 187.452 0)
 			(effects
@@
 			)
 		)
-		(property "Value" "1N4148WS"
+		(property "Value" "1N4148WT"
 			(at 392.557 96.012 0)
 			(effects
@@
 			)
 		)
-		(property "Value" "1N4148WS"
+		(property "Value" "1N4148WT"
 			(at 193.167 97.282 0)
 			(effects
@@
 			)
 		)
-		(property "Value" "1N4148WS"
+		(property "Value" "1N4148WT"
 			(at 293.497 42.672 0)
 			(effects
@@
 			)
 		)
-		(property "Value" "1N4148WS"
+		(property "Value" "1N4148WT"
 			(at 294.767 96.012 0)
 			(effects
@@
 			)
 		)
-		(property "Value" "1N4148WS"
+		(property "Value" "1N4148WT"
 			(at 264.668 38.862 0)
 			(effects
@@
 			)
 		)
-		(property "Value" "1N4148WS"
+		(property "Value" "1N4148WT"
 			(at 490.347 136.652 0)
 			(effects
@@
 			)
 		)
-		(property "Value" "1N4148WS"
+		(property "Value" "1N4148WT"
 			(at 490.347 94.742 0)
 			(effects
@@
 			)
 		)
-		(property "Value" "1N4148WS"
+		(property "Value" "1N4148WT"
 			(at 393.827 47.752 0)
 			(effects
@@
 			)
 		)
-		(property "Value" "1N4148WS"
+		(property "Value" "1N4148WT"
 			(at 293.497 182.372 0)
 			(effects
@@
 			)
 		)
-		(property "Value" "1N4148WS"
+		(property "Value" "1N4148WT"
 			(at 360.172 176.784 0)
 			(effects
@@
 			)
 		)
-		(property "Value" "1N4148WS"
+		(property "Value" "1N4148WT"
 			(at 263.652 177.292 0)
 			(effects
@@
 			)
 		)
-		(property "Value" "1N4148WS"
+		(property "Value" "1N4148WT"
 			(at 360.68 36.576 0)
 			(effects
@@
 			)
 		)
-		(property "Value" "1N4148WS"
+		(property "Value" "1N4148WT"
 			(at 395.097 181.102 0)
 			(effects
@@
 			)
 		)
-		(property "Value" "1N4148WS"
+		(property "Value" "1N4148WT"
 			(at 262.636 85.852 0)
 			(effects
@@
 			)
 		)
-		(property "Value" "1N4148WS"
+		(property "Value" "1N4148WT"
 			(at 193.167 92.202 0)
 			(effects
@@
 			)
 		)
-		(property "Value" "1N4148WS"
+		(property "Value" "1N4148WT"
 			(at 293.497 143.002 0)
 			(effects
@@
 			)
 		)
-		(property "Value" "1N4148WS"
+		(property "Value" "1N4148WT"
 			(at 393.827 140.462 0)
 			(effects
@@
 			)
 		)
-		(property "Value" "1N4148WS"
+		(property "Value" "1N4148WT"
 			(at 193.167 50.292 0)
 			(effects
@@
 			)
 		)
-		(property "Value" "1N4148WS"
+		(property "Value" "1N4148WT"
 			(at 490.347 41.402 0)
 			(effects
@@
 			)
 		)
-		(property "Value" "1N4148WS"
+		(property "Value" "1N4148WT"
 			(at 260.858 130.81 0)
 			(effects
@@
 			)
 		)
-		(property "Value" "1N4148WS"
+		(property "Value" "1N4148WT"
 			(at 393.827 135.382 0)
 			(effects
@@
 			)
 		)
-		(property "Value" "1N4148WS"
+		(property "Value" "1N4148WT"
 			(at 301.498 367.157 0)
 			(effects
@@
 			)
 		)
-		(property "Value" "1N4148WS"
+		(property "Value" "1N4148WT"
 			(at 193.167 45.212 0)
 			(effects

Commit message: Fixed Circuits
Parts:
- removed C58, C59, C60, C61, C62, C63, C64, C65, C66, C67, C68, C69, C70, C71, C72, C73: 33n, Capacitor_SMD:C_0603_1608Metric, symbol LrE-6-rescue:C-Device
- removed D17, D18, D19, D20, D21, D22, D23, D24, D25, D26, D27, D28, D29, D30, D31, D32, D33, D34, D35, D36, D37, D38, D39, D40, D41, D42, D43, D44, D45, D46, D47, D48: 1N4148WT, Diode_SMD:D_SOD-523, symbol LrE-6-rescue:1N4148W-Diode
- removed J2: Conn_02x05_Odd_Even, Connector_PinHeader_1.27mm:PinHeader_2x05_P1.27mm_Horizontal, symbol Connector_Generic:Conn_02x05_Odd_Even
- removed R1, R10, R11, R12, R13, R14, R15, R16, R17, R18, R19, R2, R20, R21, R22, R23, R24, R25, R26, R27, R28, R29, R3, R30, R31, R32, R4, R5, R6, R7, R8, R9: 10K, Resistor_SMD:R_0603_1608Metric, symbol LrE-6-rescue:R-Device
- removed R40, R41, R42, R43, R44, R45, R46, R47, R48, R49, R50, R51, R52, R53, R54, R55: 1K, Resistor_SMD:R_0603_1608Metric, symbol Device:R
- removed U1: STM32F072C8Tx, Package_QFP:LQFP-48_7x7mm_P0.5mm, symbol LrE-6-rescue:STM32F072C8Tx-MCU_ST_STM32F0
- added C40: 4.7u, Capacitor_SMD:C_0805_2012Metric, symbol LrE-6-rescue:C-Device
- added C41: 100n, Capacitor_SMD:C_0603_1608Metric, symbol LrE-6-rescue:C-Device
- added J2: Conn_02x07_Odd_Even, symbol Connector_Generic:Conn_02x07_Odd_Even
- added R42, R43, R44, R45: 1K, Resistor_SMD:R_0603_1608Metric, symbol LrE-6-rescue:R-Device
- added U1: STM32F072R8Tx, Package_QFP:LQFP-64_10x10mm_P0.5mm, symbol MCU_ST_STM32F0:STM32F072R8Tx
- C38: value 33n -> 4.7u; footprint Capacitor_SMD:C_0603_1608Metric -> Capacitor_SMD:C_0805_2012Metric
- R1: renamed from R60; value 1K -> 10K
- R10: renamed from R69; value 1K -> 10K
- R11: renamed from R70; value 1K -> 10K
- R12: renamed from R71; value 1K -> 10K
- R13: renamed from R72; value 1K -> 10K
- R14: renamed from R73; value 1K -> 10K
- R15: renamed from R74; value 1K -> 10K
- R16: renamed from R75; value 1K -> 10K
- R17: renamed from R76; value 1K -> 10K
- R18: renamed from R77; value 1K -> 10K
- R19: renamed from R78; value 1K -> 10K
- R2: renamed from R61; value 1K -> 10K
- R20: renamed from R79; value 1K -> 10K
- R21: renamed from R80; value 1K -> 10K
- R22: renamed from R81; value 1K -> 10K
- R23: renamed from R82; value 1K -> 10K
- R24: renamed from R83; value 1K -> 10K
- R25: renamed from R84; value 1K -> 10K
- R26: renamed from R85; value 1K -> 10K
- R27: renamed from R86; value 1K -> 10K
- R28: renamed from R87; value 1K -> 10K
- R29: renamed from R88; value 1K -> 10K
- R3: renamed from R62; value 1K -> 10K
- R30: renamed from R89; value 1K -> 10K
- R31: renamed from R90; value 1K -> 10K
- R32: renamed from R91; value 1K -> 10K
- R33: renamed from R38; footprint Resistor_SMD:R_0603_1608Metric -> Resistor_SMD:R_0805_2012Metric
- R37: renamed from R35; value 470 -> 330
- R39: renamed from R56; footprint Resistor_SMD:R_0603_1608Metric -> Resistor_SMD:R_0805_2012Metric
- R4: renamed from R63; value 1K -> 10K
- R40: renamed from R39; footprint Resistor_SMD:R_0603_1608Metric -> Resistor_SMD:R_0805_2012Metric
- R41: renamed from R36; footprint Resistor_SMD:R_0603_1608Metric -> Resistor_SMD:R_0805_2012Metric
- R5: renamed from R64; value 1K -> 10K
- R6: renamed from R65; value 1K -> 10K
- R7: renamed from R66; value 1K -> 10K
- R8: renamed from R67; value 1K -> 10K
- R9: renamed from R68; value 1K -> 10K
- renumbered C40 to C33, C41 to C35, C42 to C36, C43 to C37, C44 to C39, C45 to C42, C46 to C43, C48 to C44, C33 to C45, C34 to C46, C35 to C47, C50 to C48, C51 to C49, C52 to C50, C53 to C51, C54 to C52, C55 to C53, C56 to C54, C57 to C55, C36 to C56, C37 to C57, C47 to C58, D50 to D17, D51 to D18, D52 to D19, D53 to D20, D54 to D21, D49 to D22, D55 to D23, D56 to D24, D57 to D25, D58 to D26, R37 to R34, R33 to R35, R34 to R36, R57 to R38, REF01 to REF1, SW20 to SW19, SW5 to SW4, SW4 to SW5
Connections:
- net M6 is gone; now on net M3: D11.1 (K)
- net M7 is gone; now on net M0: D12.1 (K)
- net M8 is gone; now on net M2: D14.1 (K)
- net M9 is gone; now on net M1: D15.1 (K)
- net +3V3: now also C38.2, R1.1, R10.1, R11.1, R12.1, R13.1, R14.1, R15.1, R16.1, R17.1, R18.1, R19.2, R2.1, R20.2, R21.2, R22.2, R23.2, R24.2, R25.1, R26.1, R27.1, R28.1, R29.1, R3.1, R30.1, R31.1, R32.1, R4.1, R5.1, R6.1, R7.1, R8.1, R9.1, C40.2, C41.2, J2.3 (Pin_3), U1.1 (VBAT), U1.13 (VDDA), U1.19 (VDD), U1.32 (VDD), U1.48 (VDDIO2), U1.64 (VDD)
- net DFU: now also U1.60 (BOOT0)
- net GND: now also C38.1, SW1.C, SW10.C, SW11.C, SW12.C, SW13.C, SW14.C, SW15.C, SW16.C, SW2.C, SW3.C, SW4.C, SW5.C, SW6.C, SW7.C, SW8.C, SW9.C, C40.1, C41.1, J2.11 (Pin_11), J2.5 (Pin_5), J2.7 (Pin_7), R42.2, R43.2, R44.2, R45.2, U1.12 (VSSA), U1.18 (VSS), U1.31 (VSS), U1.47 (VSS), U1.63 (VSS); no longer C38.2, R1.2, R10.2, R11.2, R12.2, R13.2, R14.2, R15.2, R16.2, R17.2, R18.2, R19.1, R2.2, R20.1, R21.1, R22.1, R23.1, R24.1, R25.2, R26.2, R27.2, R28.2, R29.2, R3.2, R30.2, R31.2, R32.2, R4.2, R5.2, R6.2, R7.2, R8.2, R9.2
- net L0: now also SW1.S1, SW2.S1, SW3.S1, SW5.S1, U1.5 (PF0)
- net L1: now also SW4.S1, SW6.S1, SW7.S1, SW8.S1, U1.6 (PF1)
- net L2: now also SW10.S1, SW11.S1, SW12.S1, SW9.S1, U1.54 (PD2)
- net LED_DON: now also U1.22 (PA6)
- net M0: now also D13.1 (K), D5.1 (K), R42.1, U1.14 (PA0); no longer D2.1 (K)
- net M1: now also D10.1 (K), D2.1 (K), D6.1 (K), R43.1, U1.15 (PA1); no longer D3.1 (K), D4.1 (K)
- net M2: now also D3.1 (K), D9.1 (K), R44.1, U1.16 (PA2); no longer D5.1 (K)
- net M3: now also D16.1 (K), D4.1 (K), D8.1 (K), R45.1, U1.17 (PA3); no longer D10.1 (K), D6.1 (K)
- net NRST: now also J2.12 (Pin_12), U1.7 (NRST)
- net SP: now also U1.41 (PA8)
- net SWCLK: now also J2.6 (Pin_6), U1.49 (PA14)
- net SWDIO: now also J2.4 (Pin_4), U1.46 (PA13)
- net USB_DM: now also U1.44 (PA11)
- net USB_DP: now also U1.45 (PA12)
- net E9A: now reaches C19.1, SW10.A
- net E9A: now also R19.1, U1.28 (PB2); no longer R19.2
- net E9B: now reaches C20.1, SW10.B
- net E9B: now also R20.1, U1.55 (PB3); no longer R20.2
- net at SW10.S2: now also D10.2 (A)
- net E10A: now reaches C21.1, SW11.A
- net E10A: now also R21.1, U1.56 (PB4); no longer R21.2
- net E10B: now reaches C22.1, SW11.B
- net E10B: now also R22.1, U1.57 (PB5); no longer R22.2
- net at SW11.S2: now also D9.2 (A)
- net E11A: now reaches C23.1, SW12.A
- net E11A: now also R23.1, U1.58 (PB6); no longer R23.2
- net E11B: now reaches C24.1, SW12.B
- net E11B: now also R24.1, U1.59 (PB7); no longer R24.2
- net at SW12.S2: now also D11.2 (A)
- net E12A: now reaches C25.1, SW13.A
- net E12A: now also R25.2, U1.61 (PB8); no longer R25.1
- net E12B: now reaches C26.1, SW13.B
- net E12B: now also R26.2, U1.62 (PB9); no longer R26.1
- net L3: now reaches SW13.S1
- net L3: now also SW14.S1, SW15.S1, SW16.S1, U1.42 (PA9)
- net at SW13.S2: now also D13.2 (A)
- net E13A: now reaches C27.1, SW14.A
- net E13A: now also R27.2, U1.29 (PB10); no longer R27.1
- net E13B: now reaches C28.1, SW14.B
- net E13B: now also R28.2, U1.30 (PB11); no longer R28.1
- net at SW14.S2: now also D15.2 (A)
- net E8A: now reaches C17.1, SW9.A
- net E8A: now also R17.2, U1.26 (PB0); no longer R17.1
- net E8B: now reaches C18.1, SW9.B
- net E8B: now also R18.2, U1.27 (PB1); no longer R18.1
- net at SW9.S2: now also D12.2 (A)
- net E14A: now reaches C29.1, SW15.A
- net E14A: now also R29.2, U1.33 (PB12); no longer R29.1
- net E14B: now reaches C30.1, SW15.B
- net E14B: now also R30.2, U1.34 (PB13); no longer R30.1
- net at SW15.S2: now also D14.2 (A)
- net E15A: now reaches C31.1, SW16.A
- net E15A: now also R31.2, U1.35 (PB14); no longer R31.1
- net E15B: now reaches C32.1, SW16.B
- net E15B: now also R32.2, U1.36 (PB15); no longer R32.1
- net at SW16.S2: now also D16.2 (A)
- net E5A: now reaches C11.1, SW6.A
- net E5A: now also R11.2, U1.51 (PC10); no longer R11.1
- net at D4.2 (A): now also SW5.S2; no longer SW2.S1
- net E2B: now reaches C6.1, SW3.B
- net E2B: now also R6.2, U1.25 (PC5); no longer D9.2 (A), R6.1
- net E2A: now reaches C5.1, SW3.A
- net E2A: now also R5.2, U1.24 (PC4); no longer D8.2 (A), R5.1
- net E7B: now reaches C16.1, SW8.B
- net E7B: now also R16.2, U1.4 (PC15); no longer R16.1
- net E3A: now reaches C7.1, SW5.A
- net E3A: now also R7.2, U1.37 (PC6); no longer D11.2 (A), R7.1
- net E3B: now reaches C8.1, SW5.B
- net E3B: now also R8.2, U1.38 (PC7); no longer D12.2 (A), R8.1
- net E6A: now reaches C13.1, SW7.A
- net E6A: now also R13.2, U1.53 (PC12); no longer R13.1
- net E6B: now reaches C14.1, SW7.B
- net E6B: now also R14.2, U1.2 (PC13); no longer R14.1
- net at SW7.S2: now also D7.2 (A)
- net at SW3.S2: now also D3.2 (A)
- net at SW8.S2: now also D8.2 (A)
- net E5B: now reaches C12.1, SW6.B
- net E5B: now also R12.2, U1.52 (PC11); no longer R12.1
- net at D1.2 (A): now also SW1.S2; no longer SW1.S1
- net E4B: now reaches C10.1, SW4.B
- net E4B: now also R10.2, U1.40 (PC9); no longer D15.2 (A), R10.1
- net E7A: now reaches C15.1, SW8.A
- net E7A: now also R15.2, U1.3 (PC14); no longer R15.1
- net E0B: now reaches C2.1, SW1.B
- net E0B: now also R2.2; no longer D3.2 (A), R2.1
- net at SW6.S2: now also D6.2 (A)
- net E4A: now reaches C9.1, SW4.A
- net E4A: now also R9.2, U1.39 (PC8); no longer D14.2 (A), R9.1
- net E1A: now reaches C3.1, SW2.A
- net E1A: now also R3.2, U1.10 (PC2), U1.8 (PC0); no longer D5.2 (A), R3.1
- net E1B: now reaches C4.1, SW2.B
- net E1B: now also R4.2, U1.11 (PC3), U1.9 (PC1); no longer D6.2 (A), R4.1
- net at SW2.S2: now also D2.2 (A)
- net at D26.2 (A), LS1.2, R38.1: no longer C38.1
- net E0A: now reaches C1.1, SW1.A
- net E0A: now also R1.2; no longer D2.2 (A), R1.1
- net at SW4.S2: now also D5.2 (A)
- removed net M4: D13.1 (K), D8.1 (K)
- removed net M5: D16.1 (K), D9.1 (K)
- net SW renamed SW17
- net SW17: now also U1.23 (PA7)
- net SW2 renamed SW18
- net SW18: now also U1.43 (PA10)
- no-connect marks 16 -> 13
Other:
- title: LrT16 F1.2 -> LrT16
- moved on the sheet: C1, C10, C11, C12, C13, C14, C15, C16, C17, C18, C19, C2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
