File: LrT16.kicad_pcb (KiCad board)
At the start: 4 copper layers, 100 x 100 mm, 198 parts, among them J1 USB_C_Receptacle_USB2.0, J2 Conn_02x05_Odd_Even, Q1 2N7002, SW1 EC11_SMD, SW10 EC11_SMD, SW11 EC11_SMD, SW12 EC11_SMD, SW13 EC11_SMD, SW14 EC11_SMD, SW15 EC11_SMD, SW16 EC11_SMD, SW17 SW_Push, SW18 SW_Push, SW2 EC11_SMD, SW20 SW_SPST, SW3 EC11_SMD, SW4 EC11_SMD, SW5 EC11_SMD, SW6 EC11_SMD, SW7 EC11_SMD, SW8 EC11_SMD, SW9 EC11_SMD, U1 STM32F072C8Tx, U2 SPX3819M5-L3-3TR

Commit message: Commit for order #3
Routing:
- net GND: track 109.7 -> 118.0 mm
Changed lines of the file:
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@@
 		(tags "resistor")
 		(property "Reference" "R36"
-			(at 0 -1.55 90)
+			(at 0 -2.15 90)
 			(layer "B.SilkS")
 			(effects
 				(font
-					(size 0.9 1)
+					(size 1 0.8)
 					(thickness 0.15)
 				)
@@
 	)
 	(segment
+		(start 136.5 106.25)
+		(end 131.25 106.25)
+		(width 0.5)
+		(layer "F.Cu")
+		(net 2)
+	)
+	(segment
 		(start 148.5 111.5)
 		(end 146.7 109.7)
@@
 	)
 	(segment
+		(start 131.25 106.25)
+		(end 130 105)
+		(width 0.5)
+		(layer "F.Cu")
+		(net 2)
+	)
+	(segment
 		(start 192.907106 144.850184)
 		(end 193.441922 145.385)
@@
 	)
 	(segment
+		(start 136.79 105.96)
+		(end 136.5 106.25)
+		(width 0.5)
+		(layer "F.Cu")
+		(net 2)
+	)
+	(segment
 		(start 193.441922 160.385)
 		(end 194.085 160.385)
@@
 		(net 2)
 	)
+	(segment
+		(start 136.79 105.1)
+		(end 136.79 105.96)
+		(width 0.5)
+		(layer "F.Cu")
+		(net 2)
+	)
 	(via
 		(at 134.5 143)
@@
 	)
 	(via
-		(at 170.7 103.3)
+		(at 170.8 103.2)
 		(size 0.6)
 		(drill 0.3)
@@
 	)
 	(segment
+		(start 134.6 104.9)
+		(end 134.7 105)
+		(width 0.254)
+		(layer "F.Cu")
+		(net 6)
+	)
+	(segment
+		(start 134.7 105)
+		(end 135.42 105)
+		(width 0.254)
+		(layer "F.Cu")
+		(net 6)
+	)
+	(segment
 		(start 150.95 114.5625)
 		(end 152.0375 114.5625)
@@
 	)
 	(segment
+		(start 135.42 105)
+		(end 135.52 105.1)
+		(width 0.254)
+		(layer "F.Cu")
+		(net 6)
+	)
+	(segment
 		(start 152.0375 114.5625)
 		(end 152.2 114.4)
@@
 	)
 	(segment
-		(start 134.8 105.1)
-		(end 134.6 104.9)
-		(width 0.254)
-		(layer "B.Cu")
-		(net 6)
-	)
-	(segment
 		(start 171.9125 102.2875)
 		(end 171.9 102.3)
@@
 	)
 	(segment
-		(start 135.52 105.1)
-		(end 134.8 105.1)
-		(width 0.254)
-		(layer "B.Cu")
-		(net 6)
-	)
-	(segment
 		(start 139.3375 108.9375)
 		(end 139.3 108.9)
@@
 			)
 		)
+	)
+	(zone
+		(net 0)
+		(net_name "")
+		(layer "F.Cu")
+		(hatch edge 0.5)
+		(connect_pads
+			(clearance 0)
+		)
+		(min_thickness 0.25)
+		(filled_areas_thickness no)
+		(keepout
+			(tracks allowed)
+			(vias allowed)
+			(pads allowed)
+			(copperpour not_allowed)
+			(footprints allowed)
+		)
+		(placement
+			(enabled no)
+			(sheetname "")
+		)
+		(fill
+			(thermal_gap 0.5)
+			(thermal_bridge_width 0.5)
+		)
+		(polygon
+			(pts
+				(xy 136.25 104.5) (xy 136.25 106.25) (xy 138.75 106.25) (xy 138.75 104.5)
+			)
+		)

Commit message: Commit #4 order (add SP)
Parts:
- added D58: 1N4148W, Diode_SMD:D_SOD-123, B.Cu at (113.7, 103.9)
- added LS1: Speaker_Crystal, LrE-6:UGCT7525AN4, F.Cu at (120.0, 105.0)
- added Q2: 2N7002, Package_TO_SOT_SMD:SOT-23, B.Cu at (120.0, 105.0)
- added R57: 100, Resistor_SMD:R_0805_2012Metric, B.Cu at (114.7, 107.4)
Connections:
- U1 pad 29: unconnected-(U1-PA8-Pad29) -> /SP
Routing:
- net /SP: track 0.00 -> 51.5 mm, vias 0 -> 2
- net Net-(D58-A): track 0.00 -> 7.20 mm, vias 0 -> 1
- net Net-(Q2-D): track 0.00 -> 4.98 mm
- net +3V3: track 33.4 -> 37.1 mm, vias 13 -> 14
- net GND: track 118.0 -> 119.2 mm, vias 147 -> 146

Commit message: Commit for final F1.0 order
Routing:
- net GND: track 119.2 -> 133.8 mm

Commit message: edit pcb pattern
Parts:
- moved C47 6.98 mm to (138.1, 102.4), turned to 90 degrees
- moved J2 2.60 mm to (133.0, 105.8)
- moved R36 0.70 mm to (139.7, 108.0)
Routing:
- net GND: track 133.8 -> 129.2 mm
- net /SWDIO: track 29.5 -> 32.7 mm
- net /SWCLK: track 31.2 -> 34.3 mm
- net /NRST: track 51.5 -> 53.0 mm
- net +3V3: track 37.1 -> 36.1 mm, vias 14 -> 13
